Commit message: updae

File: src/4ws_description/ros2_control/4ws.ros2_control.xacro (robot description, xacro)
@@ -10,4 +10,12 @@
       </hardware>
       <joint name="joint1">
+        <param name="id">10</param>
+        <command_interface name="position"/>
+        <command_interface name="velocity"/>
+        <state_interface name="position"/>
+        <state_interface name="velocity"/>
+        <state_interface name="effort"/>
+      </joint>
+      <joint name="joint2">
         <param name="id">11</param>
         <command_interface name="position"/>
@@ -17,5 +25,5 @@
         <state_interface name="effort"/>
       </joint>
-      <joint name="joint2">
+      <joint name="joint3">
         <param name="id">12</param>
         <command_interface name="position"/>
@@ -25,14 +33,6 @@
         <state_interface name="effort"/>
       </joint>
-      <joint name="joint3">
+      <joint name="joint4">
         <param name="id">13</param>
-        <command_interface name="position"/>
-        <command_interface name="velocity"/>
-        <state_interface name="position"/>
-        <state_interface name="velocity"/>
-        <state_interface name="effort"/>
-      </joint>
-      <joint name="joint4">
-        <param name="id">14</param>
         <command_interface name="position"/>
         <command_interface name="velocity"/>
