Commit message: update

File: src/four_ws_description/ros2_control/fourws.ros2_control.xacro (robot description, xacro)
@@ -1,5 +1,5 @@
 <?xml version="1.0"?>
 <robot xmlns:xacro="http://www.ros.org/wiki/xacro">
-  <xacro:macro name="open_manipulator_x_ros2_control" params="name">
+  <xacro:macro name="fourws_ros2_control" params="name">
     <ros2_control name="${name}" type="system">
       <hardware>

File: src/four_ws_description/ros2_control/fourws.ros2_control_gazebo.xacro (robot description, xacro)
@@ -1,5 +1,5 @@
 <?xml version="1.0"?>
 <robot xmlns:xacro="http://www.ros.org/wiki/xacro">
-  <xacro:macro name="open_manipulator_x_ros2_control" params="name">
+  <xacro:macro name="fourws_ros2_control" params="name">
     <ros2_control name="${name}" type="system">
       <hardware>
