Commit message: update

File: src/four_ws_description/ros2_control/four_ws.ros2_control.xacro (robot description, xacro)
@@ -1,5 +1,5 @@
 <?xml version="1.0"?>
 <robot xmlns:xacro="http://www.ros.org/wiki/xacro">
-  <xacro:macro name="fourws_ros2_control" params="name">
+  <xacro:macro name="four_ws_ros2_control" params="name">
     <ros2_control name="${name}" type="system">
       <hardware>
